File: pi_max31328.kicad_pcb (KiCad board)
At the start: 2 copper layers, 21.3 x 14 mm, 9 parts, among them J1 PINHD_1x5_Female, U1 MAX31328NELB+

Commit message: kicad 10
Parts:
- C1, C2, C3, C4: footprint Capacitor_SMD:C_0402_1005Metric_Pad0.74x0.62mm_HandSolder -> Capacitor_SMD:C_0805_2012Metric
- R1, R2: footprint PCM_Resistor_SMD_AKL:R_0402_1005Metric_Pad0.72x0.64mm_HandSolder -> PCM_JLCPCB:R_0805
- moved C1 2.46 mm to (26.2, 31.8)
- moved C3 2.43 mm to (26.2, 22.2)
- moved R1 1.02 mm to (28.1, 28.9)
- moved C2 0.97 mm to (22.3, 31.8)
- moved C4 0.92 mm to (22.3, 22.2)
- moved R2 0.60 mm to (28.1, 25.4), turned to -90 degrees
Connections:
- R2 pad 1: /SDA -> /VCC
- R2 pad 2: /VCC -> /SDA
Routing:
- net /VCC: track 0.00 -> 13.9 mm, vias 0 -> 1
- net /GND: track 14.0 -> 15.0 mm, vias 3 -> 4
- net /SCL: track 11.8 -> 12.8 mm
- net /SDA: track 10.4 -> 11.1 mm
Other:
- board text added: "+"
- board text added: "-"
- board text added: "4K7 4K7"
- board text added: "CR927/CR1025"
- board text added: "MAX31328 for Raspberry Pi v0.3b CC0 OSHW"
- board text added: "VBATT0.1uF1uF"
- board text added: "VCC0.1uF1uF"
- board text removed: "I2C 4.7K 4.7K"
- board text removed: "MAX31328 for Raspberry Pi v0.2 CC0 OSHW"
- board text removed: "VBATT 0.1uF 1uF"
- board text removed: "VCC 0.1uF 1uF"
