File: pi_max31328.kicad_sch (KiCad schematic)
At the start: 9 parts, among them J1 PINHD_1x5_Female, U1 MAX31328NELB+

Commit message: kicad 10
Parts:
- C1, C2, C3, C4: footprint PCM_Capacitor_SMD_AKL:C_0402_1005Metric -> PCM_Capacitor_SMD_AKL:C_0805_2012Metric; symbol Device:C -> PCM_Capacitor_AKL:C_0805
- J1: symbol PCM_SL_Pin_Headers:PINHD_1x5_Female -> Connector:Conn_01x05_Socket
- R1, R2: footprint PCM_Resistor_SMD_AKL:R_0402_1005Metric -> PCM_Resistor_SMD_AKL:R_0805_2012Metric; symbol PCM_Resistor_AKL:R_0402 -> PCM_Resistor_AKL:R_0805
Connections:
- net SDA: now also R2.2; no longer R2.1
- net VCC: now also R2.1; no longer R2.2
Other:
- moved on the sheet: BAT1, R1, R2
